Commit message: Add files via upload

File: catkin_ws/src/lab2/urdf/Henio-robot.urdf (robot description, URDF)
Before this commit: robot Henio-robot, 5 links, 4 joints
Links:
- link czlon_1: geometry visual box size=${props[3]['l_len']} 0.1 0.1
- link czlon_2: geometry visual box size=0.3 0.05 0.05
- link joint_1: geometry visual sphere radius=0.1
Joints:
- joint 1_na_boki: origin xyz=0 0 0 -> xyz=${props[1]['j_xyz']} rpy=${props[1]['j_rpy']}
- joint 1_przod_tyl: axis 0 1 0 -> 0 0 1; origin xyz=0 0 0 -> xyz=${props[2]['j_xyz']} rpy=${props[2]['j_rpy']}
- joint 2 z czlonem: origin xyz=0 0 0 -> xyz=0 0 0 rpy=0 0 0
- joint czlon_z_2: axis 0 1 0 -> 0 0 1; origin xyz=0 0 0.5 -> xyz=${props[3]['j_xyz']} rpy=${props[3]['j_rpy']}
